Commit message: cartographer config done, basic features done, pending tuning

File: src/simulation/urdf/simulation.urdf (robot description, URDF)
Before this commit: robot simulation, 9 links, 8 joints
Links:
- added link dummy_base_link, mass 3.604; collision mesh filename=package://simulation/meshes/base_link.STL; visual mesh filename=package://simulation/meshes/base_link.STL
- link base_link: mass 3.604 -> None; geometry 
Joints:
- added joint base_to_dummy_base: type fixed, parent base_link, child dummy_base_link, origin xyz=0 0 0 rpy=-1.57079632 0 0
- joint cam: parent base_link -> dummy_base_link
- joint fl: parent base_link -> dummy_base_link
- joint fr: parent base_link -> dummy_base_link
- joint rad: parent base_link -> dummy_base_link
- joint ras: parent base_link -> dummy_base_link
- joint rl: parent base_link -> dummy_base_link
- joint rr: parent base_link -> dummy_base_link
